File: eagle_design_files/main_PCB/V2/mk312_smt_main_V2a.brd (EAGLE design)
At the start: 190.5 x 66 mm, 129 parts, among them IC1 MEGA16-A, J11 Z-S311024S1GK1A, J2 REMOTE INPUT, J3 LINK INPUT, J4 MIC INPUT, J5 LINE INPUT, J6 OUTPUT A, J7 OUTPUT B, J8 VDC INPUT, J9 X6511FV-06-C85D32, Q1 N-HEXFET-2D_SOT232-IRLL2705, Q2 N-HEXFET-2D_SOT232-IRLL2705, Q3 BSP170PH6327, Q4 N-HEXFET-2D_SOT232-IRLL2705, Q5 N-HEXFET-2D_SOT232-IRLL2705, Q6 BSP170PH6327, U10 LM358DR2G, U2 LM324DT, U4 LM358DR2G, U9 MAX232ESE+T, Y2 8MHZ

Commit message: Add files via upload
Parts:
- S5: device switch:LPV-1 -> MK312parts:LPV-1
Routing:
- net N$9: track 39.7 -> 42.9 mm
Changed lines of the file:
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@@
 <attribute name="VALUE" x="152.5" y="39.85" size="1.27" layer="27" ratio="10" rot="R90"/>
 </element>
-<element name="S5" library="switch" package="LPV-1" value="POWER" x="182.88" y="40.64" smashed="yes">
+<element name="S5" library="MK312parts" package="LPV-1" package3d_urn="urn:adsk.eagle:package:27681/1" value="POWER" x="182.88" y="40.64" smashed="yes">
 <attribute name="NAME" x="177.927" y="40.767" size="1.27" layer="25" ratio="10" rot="R90"/>
+<attribute name="POPULARITY" value="0" x="182.88" y="40.64" size="1.778" layer="27" display="off"/>
 <attribute name="VALUE" x="188.849" y="40.767" size="1.27" layer="27" ratio="10" rot="R90"/>
 </element>
@@
 <contactref element="S5" pad="3"/>
 <contactref element="D4" pad="C"/>
-<wire x1="182.9" y1="63" x2="182.9" y2="58.5" width="0.3048" layer="16"/>
-<wire x1="182.9" y1="58.5" x2="182.88" y2="58.42" width="0.3048" layer="16"/>
-<wire x1="182.9" y1="63" x2="182.88" y2="63.5" width="0.3048" layer="16"/>
-<wire x1="187.198" y1="65.024" x2="187.198" y2="85.693" width="1.016" layer="1"/>
+<wire x1="187.198" y1="62.87654375" x2="187.198" y2="85.693" width="1.016" layer="1"/>
 <wire x1="187.198" y1="85.693" x2="187.039" y2="85.852" width="0.8128" layer="1"/>
-<wire x1="182.88" y1="63.5" x2="185.674" y2="63.5" width="1.016" layer="1"/>
-<wire x1="185.674" y1="63.5" x2="187.198" y2="65.024" width="1.016" layer="1"/>
+<wire x1="187.198" y1="62.87654375" x2="185.0898" y2="60.96" width="1.016" layer="1"/>
+<wire x1="182.88" y1="60.96" x2="185.0898" y2="60.96" width="1.016" layer="1"/>
 <contactref element="F1" pad="2"/>
-<wire x1="182.88" y1="63.5" x2="180.086" y2="63.5" width="1.016" layer="1"/>
-<wire x1="179.197" y1="64.389" x2="179.197" y2="69.124" width="1.016" layer="1"/>
-<wire x1="180.086" y1="63.5" x2="179.197" y2="64.389" width="1.016" layer="1"/>
+<wire x1="182.88" y1="60.96" x2="180.6575" y2="60.96" width="1.016" layer="1"/>
+<wire x1="180.6575" y1="60.96" x2="179.197" y2="62.287725" width="1.016" layer="1"/>
+<wire x1="179.197" y1="62.287725" x2="179.197" y2="69.124" width="1.016" layer="1"/>
+<wire x1="182.88" y1="60.96" x2="182.88" y2="57.15" width="1.016" layer="16"/>
 </signal>
 </signals>
