File: eagle_design_files/main_PCB/V2/mk312_smt_main_V2a.sch (EAGLE design)
At the start: 129 parts, among them IC1 MEGA16-A, J11 Z-S311024S1GK1A, J2 REMOTE INPUT, J3 LINK INPUT, J4 MIC INPUT, J5 LINE INPUT, J6 OUTPUT A, J7 OUTPUT B, J8 VDC INPUT, J9 X6511FV-06-C85D32, Q1 N-HEXFET-2D_SOT232-IRLL2705, Q2 N-HEXFET-2D_SOT232-IRLL2705, Q3 BSP170PH6327, Q4 N-HEXFET-2D_SOT232-IRLL2705, Q5 N-HEXFET-2D_SOT232-IRLL2705, Q6 BSP170PH6327, U10 LM358DR2G, U2 LM324DT, U4 LM358DR2G, U9 MAX232ESE+T, Y2 8MHZ

Commit message: Add files via upload
Parts:
- S5: device switch:LPV-1 -> MK312parts:LPV-1
Changed lines of the file:
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@@
 <part name="GND21" library="supply2" deviceset="GND" device=""/>
 <part name="GND40" library="supply2" deviceset="GND" device=""/>
-<part name="S5" library="switch" deviceset="LPV-1" device="" value="POWER"/>
+<part name="S5" library="MK312parts" deviceset="LPV-1" device="" package3d_urn="urn:adsk.eagle:package:27681/1" value="POWER"/>
 <part name="GND42" library="supply2" deviceset="GND" device=""/>
 <part name="GND29" library="supply2" deviceset="GND" device=""/>
