File: LiFePO4_Charger/LiFePO4_Charger.brd (EAGLE design)
At the start: 38.3 x 22.8 mm, 20 parts, among them U1 MP2759

Commit message: Add files via upload
Connections:
- removed net N$10: R2.1, U$1.P$2
- net N$7: now also R2.1, U$1.P$2
Routing:
- net N$7: track 0.00 -> 28.0 mm
- net N$10: track 14.6 -> 0.00 mm
Changed lines of the file:
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@@
 <signal name="N$7">
 <contactref element="U1" pad="15"/>
+<contactref element="R2" pad="1"/>
+<contactref element="U$1" pad="P$2"/>
+<wire x1="24.765" y1="19.964" x2="23.647" y2="19.964" width="0.508" layer="1"/>
+<wire x1="23.647" y1="19.964" x2="22.86" y2="19.177" width="0.508" layer="1"/>
+<wire x1="22.86" y1="19.177" x2="22.86" y2="15.113" width="0.508" layer="1"/>
+<wire x1="25.149" y1="12.824" x2="22.86" y2="15.113" width="0.508" layer="1"/>
+<wire x1="25.149" y1="12.824" x2="30.226" y2="12.824" width="0.508" layer="1"/>
+<wire x1="12.919" y1="11.684" x2="12.919" y2="11.303" width="0.3048" layer="1"/>
+<wire x1="15.621" y1="13.97" x2="17.653" y2="13.97" width="0.3048" layer="1"/>
+<wire x1="19.431" y1="13.97" x2="21.59" y2="13.97" width="0.3048" layer="1"/>
+<wire x1="22.733" y1="15.113" x2="22.86" y2="15.113" width="0.3048" layer="1"/>
+<wire x1="21.59" y1="13.97" x2="21.717" y2="14.097" width="0.3048" layer="1"/>
+<wire x1="12.919" y1="10.544" x2="12.919" y2="11.303" width="0.2032" layer="1"/>
+<wire x1="21.717" y1="14.097" x2="22.733" y2="15.113" width="0.508" layer="1"/>
+<wire x1="12.919" y1="13.173" x2="13.716" y2="13.97" width="0.508" layer="1"/>
+<wire x1="12.919" y1="13.173" x2="12.919" y2="11.684" width="0.508" layer="1"/>
+<wire x1="13.716" y1="13.97" x2="15.621" y2="13.97" width="0.508" layer="1"/>
+<wire x1="17.653" y1="13.97" x2="19.431" y2="13.97" width="0.508" layer="1"/>
 </signal>
 <signal name="BAT_IN" class="2">
@@
 <contactref element="C5" pad="2"/>
 <via x="27.559" y="15.24" extent="1-16" drill="0.35" shape="octagon"/>
-<via x="13.716" y="12.065" extent="1-16" drill="0.35" shape="octagon"/>
-<wire x1="13.469" y1="10.294" x2="13.469" y2="11.818" width="0.2" layer="1"/>
-<wire x1="13.469" y1="11.818" x2="13.716" y2="12.065" width="0.2" layer="1"/>
-<wire x1="13.716" y1="12.065" x2="24.384" y2="12.065" width="0.508" layer="16"/>
+<via x="13.843" y="12.065" extent="1-16" drill="0.35" shape="octagon"/>
+<wire x1="13.469" y1="10.294" x2="13.469" y2="11.691" width="0.2" layer="1"/>
+<wire x1="13.469" y1="11.691" x2="13.843" y2="12.065" width="0.2" layer="1"/>
+<wire x1="13.843" y1="12.065" x2="24.384" y2="12.065" width="0.508" layer="16"/>
 <wire x1="24.384" y1="12.065" x2="27.559" y2="15.24" width="0.508" layer="16"/>
 <contactref element="BAT" pad="1"/>
@@
 <wire x1="27.559" y1="17.084" x2="27.559" y2="15.24" width="0.508" layer="1"/>
 <contactref element="SV1" pad="3"/>
-<wire x1="1.905" y1="10.414" x2="12.065" y2="10.414" width="0.508" layer="16"/>
-<wire x1="12.065" y1="10.414" x2="13.716" y2="12.065" width="0.508" layer="16"/>
+<wire x1="1.905" y1="10.414" x2="12.192" y2="10.414" width="0.508" layer="16"/>
+<wire x1="12.192" y1="10.414" x2="13.843" y2="12.065" width="0.508" layer="16"/>
 </signal>
 <signal name="N$2">
@@
 <wire x1="18.034" y1="18.669" x2="19.089" y2="18.669" width="0.3048" layer="1"/>
 <wire x1="19.089" y1="18.669" x2="19.939" y2="17.819" width="0.3048" layer="1"/>
-</signal>
-<signal name="N$10">
-<contactref element="R2" pad="1"/>
-<contactref element="U$1" pad="P$2"/>
-<wire x1="24.765" y1="19.964" x2="23.647" y2="19.964" width="0.508" layer="1"/>
-<wire x1="23.647" y1="19.964" x2="22.86" y2="19.177" width="0.508" layer="1"/>
-<wire x1="22.86" y1="19.177" x2="22.86" y2="15.113" width="0.508" layer="1"/>
-<wire x1="22.86" y1="15.113" x2="25.149" y2="12.824" width="0.508" layer="1"/>
-<wire x1="25.149" y1="12.824" x2="30.226" y2="12.824" width="0.508" layer="1"/>
 </signal>
 <signal name="VCC">
@@
 <contactref element="R6" pad="1"/>
 <contactref element="U1" pad="13"/>
-<via x="14.732" y="13.208" extent="1-16" drill="0.35" shape="octagon"/>
+<via x="14.732" y="13.081" extent="1-16" drill="0.35" shape="octagon"/>
 <via x="14.732" y="17.78" extent="1-16" drill="0.35" shape="octagon"/>
 <wire x1="14.732" y1="17.78" x2="14.771" y2="17.819" width="0.254" layer="1"/>
@@
 <wire x1="14.732" y1="10.541" x2="14.732" y2="10.16" width="0.2" layer="1"/>
 <wire x1="14.316" y1="9.744" x2="14.732" y2="10.16" width="0.2" layer="1"/>
-<wire x1="14.732" y1="17.78" x2="14.732" y2="13.208" width="0.508" layer="16"/>
-<wire x1="14.732" y1="13.208" x2="14.732" y2="10.541" width="0.3048" layer="1"/>
+<wire x1="14.732" y1="17.78" x2="14.732" y2="13.081" width="0.508" layer="16"/>
+<wire x1="14.732" y1="13.081" x2="14.732" y2="10.541" width="0.3048" layer="1"/>
 </signal>
 <signal name="N$14">

Commit message: Add files via upload
Parts:
- removed U$1: 22uH, MK312parts:SMDRI129-220MT
- added L1: 10uH, MK312parts:FXL0630-100-M
- moved C5 6.17 mm to (24.3, 12.8), turned to 90 degrees
- moved BAT 4.70 mm to (29.3, 18.0), turned to 270 degrees
- moved R2 0.52 mm to (24.3, 18.7)
Connections:
- net N$7: now also L1.P$2; no longer U$1.P$2
- net SW: now also L1.P$1; no longer U$1.P$1
Routing:
- net N$7: track 28.0 -> 41.7 mm
- net BAT_IN: track 46.0 -> 37.9 mm
- net SW: track 28.7 -> 25.2 mm
Other:
- board size 38.3 x 22.8 mm -> 33 x 22.8 mm
