File: LiFePO4_Charger/LiFePO4_Charger.sch (EAGLE design)
At the start: 20 parts, among them U1 MP2759

Commit message: Add files via upload
Connections:
- removed net N$10: R2.1, U$1.2
- net N$7: now also R2.1, U$1.2
Changed lines of the file:
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@@
 <net name="N$7" class="0">
 <segment>
-<junction x="190.5" y="121.92"/>
 <pinref part="U1" gate="G$1" pin="CSP"/>
 <wire x1="149.86" y1="116.84" x2="190.5" y2="116.84" width="0.1524" layer="91"/>
-<wire x1="190.5" y1="121.92" x2="190.5" y2="116.84" width="0.1524" layer="91"/>
+<pinref part="R2" gate="G$1" pin="1"/>
+<pinref part="U$1" gate="G$1" pin="2"/>
+<wire x1="187.96" y1="121.92" x2="190.5" y2="121.92" width="0.1524" layer="91"/>
+<wire x1="190.5" y1="121.92" x2="193.04" y2="121.92" width="0.1524" layer="91"/>
+<wire x1="190.5" y1="116.84" x2="190.5" y2="121.92" width="0.1524" layer="91"/>
+<junction x="190.5" y="121.92"/>
 </segment>
 </net>
@@
 </segment>
 </net>
-<net name="N$10" class="0">
-<segment>
-<pinref part="R2" gate="G$1" pin="1"/>
-<pinref part="U$1" gate="G$1" pin="2"/>
-<wire x1="187.96" y1="121.92" x2="193.04" y2="121.92" width="0.1524" layer="91"/>
-</segment>
-</net>

Commit message: Add files via upload
Parts:
- removed U$1: 22uH, MK312parts:SMDRI129-220MT
- added L1: 10uH, MK312parts:FXL0630-100-M
Connections:
- net N$7: now also L1.2; no longer U$1.2
- net SW: now also L1.1; no longer U$1.1
Changed lines of the file:
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@@
 <part name="SUPPLY2" library="supply2" library_urn="urn:adsk.eagle:library:372" deviceset="GND" device=""/>
 <part name="SUPPLY3" library="supply2" library_urn="urn:adsk.eagle:library:372" deviceset="GND" device=""/>
-<part name="U$1" library="MK312parts" deviceset="SMDRI129-220MT" device="" value="22uH"/>
+<part name="L1" library="MK312parts" deviceset="FXL0630-100-M" device="" value="10uH"/>
 <part name="C1" library="rcl" library_urn="urn:adsk.eagle:library:334" deviceset="C-EU" device="C0805" package3d_urn="urn:adsk.eagle:package:23617/2" value="100nF"/>
 <part name="C2" library="rcl" library_urn="urn:adsk.eagle:library:334" deviceset="C-EU" device="C0805" package3d_urn="urn:adsk.eagle:package:23617/2" value="1uF"/>
@@
 <attribute name="VALUE" x="98.933" y="80.645" size="1.778" layer="96"/>
 </instance>
-<instance part="U$1" gate="G$1" x="182.88" y="121.92" smashed="yes">
+<instance part="L1" gate="G$1" x="182.88" y="121.92" smashed="yes">
 <attribute name="NAME" x="179.07" y="123.4186" size="1.778" layer="95"/>
 <attribute name="VALUE" x="179.07" y="118.618" size="1.778" layer="96"/>
@@
 <segment>
 <pinref part="U1" gate="G$1" pin="SW"/>
-<pinref part="U$1" gate="G$1" pin="1"/>
+<pinref part="L1" gate="G$1" pin="1"/>
 <wire x1="149.86" y1="121.92" x2="165.1" y2="121.92" width="0.1524" layer="91"/>
 <pinref part="C1" gate="G$1" pin="2"/>
@@
 <wire x1="149.86" y1="116.84" x2="190.5" y2="116.84" width="0.1524" layer="91"/>
 <pinref part="R2" gate="G$1" pin="1"/>
-<pinref part="U$1" gate="G$1" pin="2"/>
+<pinref part="L1" gate="G$1" pin="2"/>
 <wire x1="187.96" y1="121.92" x2="190.5" y2="121.92" width="0.1524" layer="91"/>
 <wire x1="190.5" y1="121.92" x2="193.04" y2="121.92" width="0.1524" layer="91"/>
